File: breadboard-helper.kicad_pcb (KiCad board)
At the start: 2 copper layers, 15 x 51 mm, 5 parts, among them J1 POWER_A_1, J2 POWER_B_1, J3 POWER_A_2, J4 POWER_B_2

Commit message: Add 1N5819HW diodes for reverse polarity protection
Parts:
- added D1: 1N5819HW, Diode_SMD:D_SOD-123, B.Cu at (150.0, 82.2)
- added D2: 1N5819HW, Diode_SMD:D_SOD-123, B.Cu at (150.0, 117.8)
Connections:
- net +12V renamed Net-(D1-A)
- net -12V renamed Net-(D2-K)
Routing:
- net Net-(D2-K): track 10.2 -> 17.4 mm
- net Net-(D1-A): track 10.2 -> 17.4 mm

Commit message: Add polarity markings
Other:
- board text added: "G"
Changed lines of the file:
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@@
     )
   )
+  (gr_line (start 143.25 76.605) (end 143.25 75.855)
+    (stroke (width 0.15) (type default)) (layer "F.SilkS"))
+  (gr_line (start 156.75 76.605) (end 156.75 75.855)
+    (stroke (width 0.15) (type default)) (layer "F.SilkS"))
+  (gr_line (start 156.375 123.77) (end 157.125 123.77)
+    (stroke (width 0.15) (type default)) (layer "F.SilkS"))
+  (gr_line (start 142.875 123.77) (end 143.625 123.77)
+    (stroke (width 0.15) (type default)) (layer "F.SilkS"))
+  (gr_line (start 156.375 76.23) (end 157.125 76.23)
+    (stroke (width 0.15) (type default)) (layer "F.SilkS"))
+  (gr_line (start 142.875 76.23) (end 143.625 76.23)
+    (stroke (width 0.15) (type default)) (layer "F.SilkS"))
   (gr_line (start 160.16 123.77) (end 139.84 123.77)
     (stroke (width 0.15) (type solid)) (layer "Eco1.User"))
@@
     (effects (font (size 1 1) (thickness 0.15)) (justify mirror))
   )
+  (gr_text "G" (at 156.75 121.23) (layer "F.SilkS")
+    (effects (font (size 1 1) (thickness 0.15)))
+  )
   (gr_text "P-XX" (at 150 122.5 90) (layer "F.SilkS")
+    (effects (font (size 1 1) (thickness 0.15)))
+  )
+  (gr_text "G" (at 143.25 121.23) (layer "F.SilkS")
+    (effects (font (size 1 1) (thickness 0.15)))
+  )
+  (gr_text "G" (at 143.25 78.77) (layer "F.SilkS")
     (effects (font (size 1 1) (thickness 0.15)))
   )
@@
     (effects (font (size 1 1) (thickness 0.15)))
   )
+  (gr_text "G" (at 156.75 78.77) (layer "F.SilkS")
+    (effects (font (size 1 1) (thickness 0.15)))
+  )
